File: IR Dis Circuit/_saved_IR Dis Circuit.sch (KiCad schematic (older format))
At the start: 5 parts

Commit message: Updated KiCad Value, tried put all code together, not working yet
Parts:
- D1: value IR 940nm -> VSLY5940 IR940nm
- R1: renamed from R?; value 980R -> 2k2
- gave numbers to parts that had none: 3
Changed lines of the file:
@@
 LIBS:valves
 LIBS:Vishay
-LIBS:Board Design-cache
 EELAYER 25 0
 EELAYER END
@@
 $EndDescr
 $Comp
-L PN2222A Q?
+L PN2222A Q1
 U 1 1 5BCEC41B
 P 3900 2250
-F 0 "Q?" H 4100 2325 50  0000 L CNN
+F 0 "Q1" H 4100 2325 50  0000 L CNN
 F 1 "PN2222A" H 4100 2250 50  0000 L CNN
 F 2 "TO_SOT_Packages_THT:TO-92_Molded_Narrow" H 4100 2175 50  0001 L CIN
@@
 P 4000 1750
 F 0 "D1" H 4000 1850 50  0000 C CNN
-F 1 "IR 940nm" H 4100 1650 50  0000 C CNN
+F 1 "VSLY5940 IR940nm" H 4100 1650 50  0000 C CNN
 F 2 "" H 4000 1750 50  0001 C CNN
 F 3 "" H 4000 1750 50  0001 C CNN
@@
 $EndComp
 $Comp
-L Conn_01x04 J?
+L Conn_01x04 J1
 U 1 1 5BCEC578
 P 2300 1650
-F 0 "J?" H 2300 1850 50  0000 C CNN
+F 0 "J1" H 2300 1850 50  0000 C CNN
 F 1 "Conn_01x04" H 2300 1350 50  0000 C CNN
 F 2 "" H 2300 1650 50  0001 C CNN
@@
 $EndComp
 $Comp
-L VCC #PWR?
+L VCC #PWR01
 U 1 1 5BCEC665
 P 2550 1400
-F 0 "#PWR?" H 2550 1250 50  0001 C CNN
+F 0 "#PWR01" H 2550 1250 50  0001 C CNN
 F 1 "VCC" H 2550 1550 50  0000 C CNN
 F 2 "" H 2550 1400 50  0001 C CNN
@@
 $EndComp
 $Comp
-L GND #PWR?
+L GND #PWR02
 U 1 1 5BCEC67F
 P 2800 1450
-F 0 "#PWR?" H 2800 1200 50  0001 C CNN
+F 0 "#PWR02" H 2800 1200 50  0001 C CNN
 F 1 "GND" H 2800 1300 50  0000 C CNN
 F 2 "" H 2800 1450 50  0001 C CNN
@@
 OUT
 $Comp
-L VCC #PWR?
+L VCC #PWR03
 U 1 1 5BCEC915
 P 3300 1400
-F 0 "#PWR?" H 3300 1250 50  0001 C CNN
+F 0 "#PWR03" H 3300 1250 50  0001 C CNN
 F 1 "VCC" H 3300 1550 50  0000 C CNN
 F 2 "" H 3300 1400 50  0001 C CNN
@@
 $EndComp
 $Comp
-L R R?
+L R R1
 U 1 1 5BCEC9A0
 P 3650 1450
-F 0 "R?" V 3730 1450 50  0000 C CNN
-F 1 "980R" V 3650 1450 50  0000 C CNN
+F 0 "R1" V 3730 1450 50  0000 C CNN
+F 1 "2k2" V 3650 1450 50  0000 C CNN
 F 2 "" V 3580 1450 50  0001 C CNN
 F 3 "" H 3650 1450 50  0001 C CNN
@@
 $EndComp
 $Comp
-L GND #PWR?
+L GND #PWR04
 U 1 1 5BCECC29
 P 4000 2550
-F 0 "#PWR?" H 4000 2300 50  0001 C CNN
+F 0 "#PWR04" H 4000 2300 50  0001 C CNN
 F 1 "GND" H 4000 2400 50  0000 C CNN
 F 2 "" H 4000 2550 50  0001 C CNN
@@
 IN
 $Comp
-L TSSP4056 U?
+L TSSP4056 U1
 U 1 1 5BCECDDA
 P 5100 1800
-F 0 "U?" H 4700 2100 50  0000 L CNN
+F 0 "U1" H 4700 2100 50  0000 L CNN
 F 1 "TSSP4056" H 4700 1500 50  0000 L CNN
 F 2 "Opto-Devices:IRReceiver_Vishay_MINICAST-3pin" H 5050 1425 50  0001 C CNN
@@
 $EndComp
 $Comp
-L VCC #PWR?
+L VCC #PWR05
 U 1 1 5BCED030
 P 5700 1500
-F 0 "#PWR?" H 5700 1350 50  0001 C CNN
+F 0 "#PWR05" H 5700 1350 50  0001 C CNN
 F 1 "VCC" H 5700 1650 50  0000 C CNN
 F 2 "" H 5700 1500 50  0001 C CNN
@@
 $EndComp
 $Comp
-L GND #PWR?
+L GND #PWR06
 U 1 1 5BCED04A
 P 5700 2200
-F 0 "#PWR?" H 5700 1950 50  0001 C CNN
+F 0 "#PWR06" H 5700 1950 50  0001 C CNN
 F 1 "GND" H 5700 2050 50  0000 C CNN
 F 2 "" H 5700 2200 50  0001 C CNN
