File: IR Dis Circuit/IR Dis Circuit.sch (KiCad schematic (older format))
At the start: 5 parts, among them J1 Conn_01x04, Q1 PN2222A, U1 TSSP4056

Commit message: Updated KiCad Value, tried put all code together, not working yet
Parts:
- D1: value IR 940nm -> VSLY5940 IR940nm
- R1: value 980R -> 820R
Changed lines of the file:
@@
 LIBS:valves
 LIBS:Vishay
-LIBS:Board Design-cache
 EELAYER 25 0
 EELAYER END
@@
 P 4000 1750
 F 0 "D1" H 4000 1850 50  0000 C CNN
-F 1 "IR 940nm" H 4100 1650 50  0000 C CNN
+F 1 "VSLY5940 IR940nm" H 4100 1650 50  0000 C CNN
 F 2 "" H 4000 1750 50  0001 C CNN
 F 3 "" H 4000 1750 50  0001 C CNN
@@
 P 3650 1450
 F 0 "R1" V 3730 1450 50  0000 C CNN
-F 1 "980R" V 3650 1450 50  0000 C CNN
+F 1 "820R" V 3650 1450 50  0000 C CNN
 F 2 "" V 3580 1450 50  0001 C CNN
 F 3 "" H 3650 1450 50  0001 C CNN

Commit message: value change
Parts:
- R1: value 820R -> 2k2
Changed lines of the file:
@@
 P 3650 1450
 F 0 "R1" V 3730 1450 50  0000 C CNN
-F 1 "820R" V 3650 1450 50  0000 C CNN
+F 1 "2k2" V 3650 1450 50  0000 C CNN
 F 2 "" V 3580 1450 50  0001 C CNN
 F 3 "" H 3650 1450 50  0001 C CNN
